File: PCB/Clock_MiniM4.kicad_pcb (KiCad board)
At the start: 2 copper layers, 132.1 x 85.7 mm, 7 parts, among them J1 5V_POWER_INPUT, M1 Feather_M4_Express, M2 Feather_M4_Express, M3 4-Bit_Level_Converter_757, U1 1.2-inch_7-segment_LED_HT16K3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

Commit message: add display I2C bias
Connections:
- U1 pad 5: (no net) -> /USB
Changed lines of the file:
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@@
   (title_block
     (title Clock_MiniM4)
-    (date 2020-03-27)
+    (date 2020-03-28)
     (rev v01)
     (company "Cedar Grove Studios")
@@
     (pad 4 thru_hole circle (at -2.54 -22.86) (size 1.524 1.524) (drill 0.762) (layers *.Cu *.Mask)
       (net 9 /USB))
-    (pad 5 thru_hole circle (at -5.08 -22.86) (size 1.524 1.524) (drill 0.762) (layers *.Cu *.Mask))
+    (pad 5 thru_hole circle (at -5.08 -22.86) (size 1.524 1.524) (drill 0.762) (layers *.Cu *.Mask)
+      (net 9 /USB))
     (pad 3 thru_hole circle (at 0 -22.86) (size 1.524 1.524) (drill 0.762) (layers *.Cu *.Mask)
       (net 1 GND))
